File: podfm.brd (EAGLE design)
At the start: 30 x 58.7 mm, 30 parts, among them IC1 ATMEGA168-AU, IC2 FT232RL, X1 MINI-USB-32005-301, X2 R141426

Commit message: 9/22/2013 fixed usb connection 1-VCC 2-data- 3-data+ 5-GND added resistor network for ipod iphone charging Signed-off-by: goose1987 <phamh1987@gmail.com>
Parts:
- added R10, R11: 10k, rcl:R1206
- moved C7 1.30 mm to (10.4, 54.4)
- moved R9 0.77 mm to (4.70, 52.1), turned to 270 degrees
- moved R8 0.76 mm to (2.54, 52.1)
- moved U$3 0.25 mm to (15.7, 55.4)
Connections:
- net GND: now also R11.2, X1.5, X1.M1, X1.M2, X1.M3, X1.M4; no longer X1.1
- net N$3: now also X1.2; no longer X1.4
- net N$7: now also R10.2, R11.1; no longer R8.1
- net N$8: now also R8.1, R9.2; no longer R9.1
- net VUSB: now also R10.1, R9.1, X1.1; no longer R9.2, X1.5
Routing:
- net VUSB: track 74.6 -> 80.1 mm
- net N$3: track 5.26 -> 10.5 mm
- net N$7: track 6.86 -> 10.3 mm, vias 1 -> 0
- net N$11: track 5.12 -> 6.60 mm
- net N$8: track 8.60 -> 9.99 mm
Other:
- board text added: "WMDM"
- board text removed: "WDMD"
